File: MH69_Data/PCB/MH69-Left/MH69-Left.kicad_pcb (KiCad board)
At the start: 2 copper layers, 164.5 x 97 mm, 77 parts, among them U1 nice_nano

Commit message: THE BIG CHANGE - schematic and PCB layout
Parts:
- removed Batt1: B+, Connector_JST:JST_PH_B2B-PH-K_1x02_P2.00mm_Vertical
- added Batt_L1: B+, Connector_PinHeader_2.54mm:PinHeader_1x02_P2.54mm_Vertical, F.Cu at (35.2, 97.2)
- added H3: MountingHole, ScottoKeebs_Scotto:Standoff_M2x6mm, F.Cu at (36.6, 119.4)
- added J1: OLED/E-Ink_L, Connector_PinHeader_2.54mm:PinHeader_1x05_P2.54mm_Vertical, F.Cu at (30.2, 90.2)
- PWR1: value POWER -> DIP_L; footprint Connector_JST:JST_PH_B2B-PH-K_1x02_P2.00mm_Vertical -> Button_Switch_SMD:SW_SPDT_PCM12
- RST1: footprint Connector_JST:JST_PH_B2B-PH-K_1x02_P2.00mm_Vertical -> Button_Switch_SMD:SW_SPST_TL3342
- U1: moved to F.Cu
- moved PWR1 52.6 mm to (26.4, 97.2), turned to 90 degrees
- moved RST1 48.7 mm to (36.2, 105.5)
- moved H6 25.9 mm to (63.5, 44.1)
- moved K_22 22.5 mm to (53.8, 118.8)
- moved K_15 22.5 mm to (53.8, 99.8)
- moved K_8 22.5 mm to (53.8, 80.8)
- moved D_15 22.5 mm to (58.5, 105.8)
- moved D_8 22.5 mm to (58.5, 86.8)
- moved D_22 22.5 mm to (58.5, 124.8)
- moved U1 19.0 mm to (35.3, 71.2), turned to -90 degrees
- moved H5 13.7 mm to (59.4, 157.7)
- moved K_0 12.0 mm to (53.8, 61.8)
- moved D_0 12.0 mm to (58.5, 67.8)
- moved H2 4.82 mm to (157.0, 71.3)
Connections:
- net Net-(RST1-A) renamed BOOT_L
- D_0 pad 1: row0 -> row0_L
- D_1 pad 1: row0 -> row0_L
- D_10 pad 1: row1 -> row1_L
- D_11 pad 1: row1 -> row1_L
- D_12 pad 1: row1 -> row1_L
- D_13 pad 1: row1 -> row1_L
- D_14 pad 1: row1 -> row1_L
- D_15 pad 1: row2 -> row2_L
- D_16 pad 1: row2 -> row2_L
- D_17 pad 1: row2 -> row2_L
- D_18 pad 1: row2 -> row2_L
- D_19 pad 1: row2 -> row2_L
- D_2 pad 1: row0 -> row0_L
- D_20 pad 1: row2 -> row2_L
- D_21 pad 1: row2 -> row2_L
- D_22 pad 1: row3 -> row3_L
- D_23 pad 1: row3 -> row3_L
- D_24 pad 1: row3 -> row3_L
- D_25 pad 1: row3 -> row3_L
- D_26 pad 1: row3 -> row3_L
- D_27 pad 1: row3 -> row3_L
- D_28 pad 1: row3 -> row3_L
- D_29 pad 1: row4 -> row4_L
- D_3 pad 1: row0 -> row0_L
- D_30 pad 1: row4 -> row4_L
- D_31 pad 1: row4 -> row4_L
- D_32 pad 1: row4 -> row4_L
- D_33 pad 1: row4 -> row4_L
- D_4 pad 1: row0 -> row0_L
- D_5 pad 1: row0 -> row0_L
- D_6 pad 1: row0 -> row0_L
- D_7 pad 1: row0 -> row0_L
- D_8 pad 1: row1 -> row1_L
- D_9 pad 1: row1 -> row1_L
- K_0 pad 1: col0 -> col0_L
- K_1 pad 1: col1 -> col1_L
- K_10 pad 1: col2 -> col2_L
- K_11 pad 1: col3 -> col3_L
- K_12 pad 1: col4 -> col4_L
- K_13 pad 1: col5 -> col5_L
- K_14 pad 1: col6 -> col6_L
- K_15 pad 1: col0 -> col0_L
- K_16 pad 1: col1 -> col1_L
- K_17 pad 1: col2 -> col2_L
- K_18 pad 1: col3 -> col3_L
- K_19 pad 1: col4 -> col4_L
- K_2 pad 1: col2 -> col2_L
- K_20 pad 1: col5 -> col5_L
- K_21 pad 1: col6 -> col6_L
- K_22 pad 1: col0 -> col0_L
- K_23 pad 1: col1 -> col1_L
- K_24 pad 1: col3 -> col3_L
- K_25 pad 1: col4 -> col4_L
- K_26 pad 1: col5 -> col5_L
- K_27 pad 1: col6 -> col6_L
- K_28 pad 1: col7 -> col7_L
- K_29 pad 1: col1 -> col1_L
- K_3 pad 1: col3 -> col3_L
- K_30 pad 1: col2 -> col2_L
- K_31 pad 1: col4 -> col4_L
- K_32 pad 1: col5 -> col5_L
- K_33 pad 1: col6 -> col6_L
- K_4 pad 1: col4 -> col4_L
- K_5 pad 1: col5 -> col5_L
- K_6 pad 1: col6 -> col6_L
- K_7 pad 1: col7 -> col7_L
- K_8 pad 1: col0 -> col0_L
- K_9 pad 1: col1 -> col1_L
- PWR1 pad 1: Net-(Batt1-Pin_2) -> VBAT
- PWR1 pad 2: Net-(PWR1-B) -> Net-(Batt_L1-Pin_1)
- RST1 pad 2: Net-(Batt1-Pin_1) -> GND
- U1 pad 1: unconnected-(U1-TX0/P0.06-Pad1) -> CS_L
- U1 pad 10: col5 -> row1_L
- U1 pad 11: col6 -> row0_L
- U1 pad 12: col7 -> unconnected-(U1-P1.06-Pad12)
- U1 pad 13: row2 -> col7_L
- U1 pad 14: row3 -> col6_L
- U1 pad 15: row4 -> col5_L
- U1 pad 16: row1 -> col4_L
- U1 pad 17: row0 -> col3_L
- U1 pad 18: unconnected-(U1-AIN0/P0.02-Pad18) -> col2_L
- U1 pad 19: unconnected-(U1-AIN5/P0.29-Pad19) -> col1_L
- U1 pad 20: unconnected-(U1-AIN7/P0.31-Pad20) -> col0_L
- U1 pad 21: unconnected-(U1-VCC-Pad21) -> VCC
- U1 pad 23: Net-(Batt1-Pin_1) -> GND
- U1 pad 24: Net-(PWR1-B) -> VBAT
- U1 pad 3: unconnected-(U1-GND-Pad3) -> GND
- U1 pad 4: unconnected-(U1-GND-Pad4) -> GND
- U1 pad 5: col0 -> SDA_L
- U1 pad 6: col1 -> SCL_L
- U1 pad 7: col2 -> row4_L
- U1 pad 8: col3 -> row3_L
- U1 pad 9: col4 -> row2_L
Routing:
- net col7_L: track 0.00 -> 294.3 mm
- net row3: track 214.6 -> 0.00 mm, vias 1 -> 0
- net col6: track 212.4 -> 0.00 mm, vias 1 -> 0
- net row1_L: track 0.00 -> 208.3 mm
- net row0: track 202.9 -> 0.00 mm
- net row0_L: track 0.00 -> 202.8 mm
- net col5: track 194.1 -> 0.00 mm
- net row1: track 186.9 -> 0.00 mm
- net col7: track 184.4 -> 0.00 mm, vias 3 -> 0
- net row2: track 182.5 -> 0.00 mm, vias 1 -> 0
- net row4: track 172.5 -> 0.00 mm, vias 1 -> 0
- net col2: track 141.7 -> 0.00 mm
- net col3: track 141.0 -> 0.00 mm, vias 1 -> 0
- net row3_L: track 0.00 -> 135.3 mm
- net col1: track 133.6 -> 0.00 mm
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Other:
- board size 164.5 x 97 mm -> 170.9 x 97 mm

Commit message: Left side finished?
Parts:
- added H7: MountingHole, ScottoKeebs_Scotto:Standoff_M2x6mm, F.Cu at (25.4, 108.3)
- moved H4 101.6 mm to (193.3, 110.3)
- moved H5 38.9 mm to (96.0, 144.4)
- moved H2 36.5 mm to (188.8, 53.3)
- moved H3 30.8 mm to (67.4, 119.3)
- moved H6 20.1 mm to (45.5, 52.9)
- moved H1 1.28 mm to (164.0, 144.4)
- moved PWR1 0.71 mm to (25.7, 97.1)
Connections:
- U1 pad 14: col6_L -> col0_L
- U1 pad 15: col5_L -> col1_L
- U1 pad 16: col4_L -> col2_L
- U1 pad 18: col2_L -> col4_L
- U1 pad 19: col1_L -> col5_L
- U1 pad 20: col0_L -> col6_L
Routing:
- net row4_L: track 95.3 -> 250.1 mm
- net col6_L: track 94.3 -> 222.6 mm, vias 0 -> 1
- net row3_L: track 135.3 -> 253.0 mm
- net col5_L: track 92.4 -> 204.3 mm, vias 0 -> 1
- net row2_L: track 126.1 -> 229.8 mm
- net col4_L: track 90.5 -> 190.1 mm
- net col3_L: track 69.8 -> 152.8 mm
- net col2_L: track 88.7 -> 155.4 mm
- net VBAT: track 0.00 -> 55.6 mm
- net BOOT_L: track 0.00 -> 54.1 mm, vias 0 -> 3
- net col1_L: track 88.1 -> 138.6 mm
- net CS_L: track 0.00 -> 38.2 mm
- net GND: track 0.00 -> 36.4 mm, vias 0 -> 2
- net col0_L: track 62.2 -> 97.0 mm
- net SDA_L: track 0.00 -> 29.4 mm
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- added copper zone on F.Cu, net GND
Other:
- board size 170.9 x 97 mm -> 171.9 x 97 mm

Commit message: Finished Left and moving on to Right
Routing:
- net GND: track 36.4 -> 12.3 mm
- net CS_L: track 38.2 -> 44.0 mm
- net SCL_L: track 25.5 -> 30.0 mm
- net BOOT_L: track 54.1 -> 51.4 mm, vias 3 -> 0
- net VBAT: track 55.6 -> 57.8 mm
- net VCC: track 28.5 -> 30.4 mm, vias 0 -> 1
- net row0_L: track 204.1 -> 205.0 mm
- net row4_L: track 250.1 -> 249.5 mm
- added copper zone on B.Cu, net (none)
- added copper zone on F.Cu, net (none)
