File: MH69_Data/PCB/MH69-Right/MH69-Right.kicad_pcb (KiCad board)
At the start: 2 copper layers, 153.8 x 92 mm, 87 parts, among them U1 nice_nano

Commit message: Finished Left and moving on to Right
Parts:
- removed K_35, K_38: KEYSW, cb:Choc-MX-19mm-2u
- removed K_36, K_39: KEYSW, cb:Choc-MX-19mm-1.5u
- removed K_37: KEYSW, cb:Choc-MX-19mm-1u
- removed K_40: KEYSW, cb:Choc-MX-19mm-2.25u
- removed K_41: KEYSW, cb:Choc-MX-19mm-1.75u
- U1: moved to F.Cu
- moved U1 293.1 mm to (368.4, 61.5), turned to -90 degrees
Connections:
- K_27 pad 1: col6 -> Net-(K_27-COL)
- K_33 pad 1: col6 -> Net-(K_27-COL)
Routing:
- net col7: track 266.7 -> 0.00 mm, vias 2 -> 0
- net col6: track 207.5 -> 0.00 mm, vias 2 -> 0
- net col5: track 200.6 -> 0.00 mm, vias 2 -> 0
- net row4: track 199.5 -> 0.00 mm, vias 5 -> 0
- net col4: track 191.4 -> 0.00 mm, vias 2 -> 0
- net col3: track 183.0 -> 0.00 mm, vias 2 -> 0
- net row3: track 163.8 -> 0.00 mm, vias 2 -> 0
- net col1: track 142.2 -> 0.00 mm
- net row2: track 142.0 -> 0.00 mm, vias 2 -> 0
- net row1: track 134.5 -> 0.00 mm
- net Net-(PWR1-A): track 124.6 -> 0.00 mm, vias 2 -> 0
- net col2: track 113.8 -> 0.00 mm
- net row0: track 112.4 -> 0.00 mm
- net Net-(RST1-B): track 99.2 -> 0.00 mm, vias 3 -> 0
- net Net-(BAT1-Pin_1): track 88.4 -> 0.00 mm, vias 3 -> 0
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Other:
- board size 153.8 x 92 mm -> 171.9 x 97 mm
