File: MH69_Data/PCB/MH69-Right/MH69-Right.kicad_sch (KiCad schematic)
At the start: 87 parts, among them U1 nice_nano

Commit message: Finished Left and moving on to Right
Parts:
- removed K_35, K_38: KEYSW, cb:Choc-MX-19mm-2u, symbol MX_Alps_Hybrid:MX-NoLED
- removed K_36, K_39: KEYSW, cb:Choc-MX-19mm-1.5u, symbol MX_Alps_Hybrid:MX-NoLED
- removed K_37: KEYSW, cb:Choc-MX-19mm-1u, symbol MX_Alps_Hybrid:MX-NoLED
- removed K_40: KEYSW, cb:Choc-MX-19mm-2.25u, symbol MX_Alps_Hybrid:MX-NoLED
- removed K_41: KEYSW, cb:Choc-MX-19mm-1.75u, symbol MX_Alps_Hybrid:MX-NoLED
- K_0, K_1, K_10, K_11, K_12, K_13, K_14, K_15, K_16, K_17, K_18, K_19, K_2, K_20, K_22, K_23, K_24, K_25, K_26, K_27, K_28, K_3, K_31, K_32, K_33, K_34, K_4, K_5, K_7, K_8, K_9: footprint cb:Choc-MX-19mm-1u -> PCM_Switch_Keyboard_Hotswap_Kailh:SW_Hotswap_Kailh_Choc_V1_Plated_1.00u
- K_21, K_29, K_30, K_6: footprint cb:Choc-MX-19mm-1.5u -> PCM_Switch_Keyboard_Hotswap_Kailh:SW_Hotswap_Kailh_Choc_V1_Plated_1.50u
Connections:
- net col6: no longer K_27.1 (COL), K_33.1 (COL)
- new net: K_27.1 (COL), K_33.1 (COL)
